File: zenith.kicad_pcb (KiCad board)
At the start: 2 copper layers, 38.3 x 41.4 mm, 82 parts, among them J1 Screw_Terminal_01x02, J2 Conn_01x03, SW1 TS-1088-AR02016, SW2 TS-1088-AR02016, U1 TPS63070RNMR, U2 BMP580, U3 BQ25883RGER, U4 ICM-45686, U5 STM32F722RETx, U6 LMR51430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

Commit message: more editing silkscreen
Parts:
- SD Card: renamed from Card1
- renumbered SW2 to BOOT, SW1 to RESET
Changed lines of the file:
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@@
 		(layer "F.Cu")
 		(at 120.46 97.32 180)
-		(property "Reference" "SW2"
+		(property "Reference" "BOOT"
 			(at 0.02 -2.09 0)
 			(layer "F.SilkS")
@@
 		(layer "F.Cu")
 		(at 129.69 73.88 180)
-		(property "Reference" "Card1"
+		(property "Reference" "SD Card"
 			(at -0.01 0 0)
 			(layer "F.SilkS")
@@
 				(font
 					(size 0.5 0.5)
-					(thickness 0.15)
+					(thickness 0.1)
+					(bold yes)
 				)
 			)
@@
 		(at 110.49 76.35)
 		(property "Reference" "U2"
-			(at -1.16 -3.1 0)
+			(at 0.22 0.32 0)
 			(layer "F.SilkS")
 			(effects
 				(font
 					(size 0.5 0.5)
-					(thickness 0.15)
+					(thickness 0.125)
 				)
 			)
@@
 		(layer "F.Cu")
 		(at 113.85 97.36)
-		(property "Reference" "SW1"
+		(property "Reference" "RESET"
 			(at 0.06 2.05 0)
 			(layer "F.SilkS")
